File: psu.kicad_pcb (KiCad board)
At the start: 2 copper layers, 100 x 100 mm, 109 parts, among them J1 METER, J3 T1A, J4 T1B, J5 T1C, J6 SENSE+, J7 SENSE-, J8 OUT+, J9 OUT-, Q1 MMBT2907A, Q10 TIP105, Q11 MMBT2907A, Q12 MMBT2907A, Q13 PMP5201Y, Q14 MMBT3904, Q15 MMBT3904, Q16 MMBT3904, Q17 MMBT2907A, Q18 PZT2222A, Q2 MMBT2907A, Q3 MMBT3904, Q4 PMP4201Y, Q5 PMP5201Y, Q6 PMP4201Y, Q7 MMBT3904, Q8 MMBT2907A, Q9 MMBT2907A

Commit message: Changed local regulator circuit, added github readme
Parts:
- removed C4: 47u 10V, IPC7351-Nominal:CAPAE660X570
- removed R12: 2k2, IPC7351-Nominal:RESC2012X50
- Q1, Q2: value MMBT2907A -> MMBT3906
- R11: value 22k -> 560
- R4, R5: value 10k -> 2k2
- R40: value 10k -> 100k
- moved C2 37.5 mm to (101.0, 66.0)
- moved D8 32.6 mm to (105.0, 102.0)
- moved DZ1 32.6 mm to (105.0, 106.0)
- moved R5 32.0 mm to (105.0, 112.0), turned to 180 degrees
- moved R4 28.1 mm to (105.0, 109.0), turned to 180 degrees
- moved R1 26.5 mm to (101.0, 106.0), turned to 90 degrees
- moved R11 21.7 mm to (105.0, 115.0), turned to 180 degrees
- moved C3 18.5 mm to (97.0, 104.0)
- moved R40 15.5 mm to (87.0, 119.0)
- moved R38 15.0 mm to (100.0, 114.0), turned to 270 degrees
- moved R37 13.5 mm to (98.0, 110.0)
- moved R39 12.0 mm to (87.0, 115.0)
- moved C11 11.7 mm to (98.0, 114.0), turned to 270 degrees
- moved Q18 9.85 mm to (92.0, 117.0), turned to 270 degrees
- moved R3 9.85 mm to (92.0, 101.0), turned to 180 degrees
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Connections:
- R11 pad 2: /V+ -> /VEE
- R4 pad 1: /VEE -> Net-(C4-Pad2)
- R4 pad 2: Net-(C4-Pad2) -> Net-(R4-Pad2)
- R40 pad 1: /VEE -> /V-
- R40 pad 2: /V- -> /VEE
- R5 pad 1: Net-(C4-Pad2) -> Net-(R4-Pad2)
- R5 pad 2: /VEE -> Net-(Q7-Pad1)
Routing:
- net /V+: track 479.7 -> 931.2 mm, vias 10 -> 48
- net (no net): track 0.00 -> 120.0 mm
- net Net-(Q7-Pad1): track 7.50 -> 28.2 mm
- net Net-(C11-Pad1): track 8.33 -> 19.5 mm
- net /VEE: track 174.1 -> 164.3 mm, vias 19 -> 16
- net Net-(C5-Pad2): track 19.9 -> 13.1 mm
- net /V-: track 195.9 -> 201.0 mm, vias 2 -> 1
- net Net-(Q1-Pad3): track 19.3 -> 14.5 mm
- net Net-(R4-Pad2): track 0.00 -> 4.71 mm
- net Net-(C3-Pad2): track 14.1 -> 9.46 mm
- net Net-(Q4-Pad4): track 14.1 -> 10.1 mm
- net Net-(Q4-Pad5): track 12.4 -> 9.71 mm
- net Net-(C4-Pad2): track 45.5 -> 43.2 mm
- net Net-(Q18-Pad3): track 8.52 -> 10.4 mm
- added copper zone on B.Cu, net /V+
- added copper zone on F.Cu, net /V+
- added copper zone on B.Cu, net /VEE
- added copper zone on F.Cu, net /VEE
- added copper zone on F.Cu, net Net-(D8-Pad3)
Other:
- board text added: "REFERENCE and LOCAL REGULATOR"
- board text added: "SETPOINT SELECTOR and BUFFER"
- board text removed: "VOLTAGE"
- board text removed: "VOLTAGE REFERENCE"

Commit message: Rev C in progress
Parts:
- removed C11: 3n3, IPC7351-Nominal:CAPC2012X70
- removed the C7 at (119.0, 65.0)
- removed the C8 at (133.0, 91.0)
- removed the D11 at (112.0, 63.5)
- removed the D12 at (112.0, 67.5)
- removed D13: MMBD4148, IPC-semi-nominal:SOT-23
- removed the D9 at (113.0, 91.5)
- removed the DS1 at (165.0, 63.5)
- removed J7: SENSE-, conn:TEST
- removed MP1, MP2, MP3, MP4: SCREW, mech:SCREW-4-SUPPORTED
- removed the Q10 at (120.0, 118.0)
- removed the Q14 at (139.5, 78.5)
- removed the Q3 at (92.0, 110.0)
- removed the Q8 at (117.0, 81.0)
- removed the R15 at (117.5, 112.0)
- removed the R26 at (150.5, 63.5)
- removed the R27 at (153.0, 63.5)
- removed the R28 at (165.0, 71.5)
- removed the R29 at (150.5, 71.5)
- removed the R37 at (98.0, 110.0)
- removed the R38 at (100.0, 114.0)
- removed the R39 at (87.0, 115.0)
- removed the R40 at (87.0, 119.0)
- removed the R9 at (108.0, 86.0)
- added C10: 1nF 1kV, IPC7351-Nominal:CAPC3216X70, F.Cu at (163.5, 128.5)
- added C4: 1n, IPC7351-Nominal:CAPC2012X70, F.Cu at (128.0, 109.0)
- added C5: 4u7, IPC7351-Nominal:CAPC3216X70, F.Cu at (135.0, 105.0)
- added D4: S1D, IPC7351-Nominal:DIOM5326X292, F.Cu at (142.5, 83.5)
- added DS2: HOT, conn:CONN_2-SIL, F.Cu at (187.5, 73.5)
- added Q18: PMP4201Y, IPC-semi-nominal:SC-70-6, F.Cu at (190.0, 92.0)
- added Q20: MMBT2907A, IPC-semi-nominal:SOT-23, F.Cu at (204.5, 75.8)
- added Q21: MMBT2907A, IPC-semi-nominal:SOT-23, F.Cu at (199.0, 71.0)
- added Q22: MMBT3904, IPC-semi-nominal:SOT-23, F.Cu at (195.0, 71.0)
- added Q4: MMBT3906, IPC-semi-nominal:SOT-23, F.Cu at (129.0, 115.0)
- added Q6: MMBT3906, IPC-semi-nominal:SOT-23, F.Cu at (135.0, 98.0)
- added Q7: PMP4201Y, IPC-semi-nominal:SC-70-6, F.Cu at (131.0, 105.0)
- added Q9: MMBT2907A, IPC-semi-nominal:SOT-23, F.Cu at (160.0, 88.0)
- added R1: 22k, IPC7351-Nominal:RESC2012X50, F.Cu at (138.0, 118.0)
- added R16: 1k, IPC7351-Nominal:RESC2012X50, F.Cu at (161.0, 95.0)
- added R17: 1k, IPC7351-Nominal:RESC2012X50, F.Cu at (163.0, 95.0)
- added R19: 1k, IPC7351-Nominal:RESC2012X50, F.Cu at (165.0, 95.0)
- added R20: 1k, IPC7351-Nominal:RESC2012X50, F.Cu at (166.5, 110.0)
- added R25: 10k, IPC7351-Nominal:RESC2012X50, F.Cu at (191.0, 100.0)
- added R30: 33, IPC7351-Nominal:RESC2012X50, F.Cu at (197.0, 92.0)
- added R41: 10k, IPC7351-Nominal:RESC2012X50, F.Cu at (195.5, 75.0)
- added R42: 100k, IPC7351-Nominal:RESC2012X50, F.Cu at (198.0, 75.0)
- added R43: 100k, conn:CONN_2-SIL, F.Cu at (179.0, 73.5)
- added R44: 270, IPC7351-Nominal:RESC2012X50, F.Cu at (195.0, 67.5)
- added R45: 1Meg, IPC7351-Nominal:RESC3216X60, F.Cu at (167.5, 128.5)
- added R5: 22k, IPC7351-Nominal:RESC2012X50, F.Cu at (132.0, 109.0)
- added R6: 18k, IPC7351-Nominal:RESC2012X50, F.Cu at (130.0, 109.0)
- added R7: 10k, IPC7351-Nominal:RESC2012X50, F.Cu at (128.0, 105.0)
- added TP1: GND, conn:TEST_SMD, F.Cu at (169.0, 89.0)
- added TP2: GND, conn:TEST_SMD, F.Cu at (158.0, 105.0)
- added TP3: GND, conn:TEST_SMD, F.Cu at (194.0, 96.5)
- added TP4: GND, conn:TEST_SMD, F.Cu at (138.5, 102.0)
- C2: value 47u -> 47u 63V; footprint passive:C-ALUM-8mm -> passive:C-ALUM-6.3mm
- C3: value 10u -> 100p; footprint IPC7351-Nominal:CAPAE530X460 -> IPC7351-Nominal:CAPC2012X70
- C6: value 33p 50V -> 47u 63V; footprint IPC7351-Nominal:RESC2012X50 -> passive:C-ALUM-6.3mm
- D1: value GBU 100V -> S1D; footprint D2 -> IPC7351-Nominal:DIOM5326X292
- D11: renamed from D14; value S1A -> S1D
- D12: renamed from D15; value S1A -> S1D
- D2, D3: value 1N4004 -> S1D; footprint semi:DO-41 -> IPC7351-Nominal:DIOM5326X292
- D5: renamed from D4; value S1A -> S1D
- D6: renamed from D5; value S1A -> S1D
- D7: renamed from D6; value S1A -> S1D
- D8: renamed from D7; value S1A -> S1D
- DS1: renamed from DS2; value LIMIT -> LIM
- J6: value SENSE+ -> SENSE; footprint conn:TEST -> conn:CONN_2-SIL
- Q13: value PMP5201Y -> MMBT2907A; footprint IPC-semi-nominal:SC-70-6 -> IPC-semi-nominal:SOT-23
- Q14: renamed from Q11; value MMBT2907A -> MMBT3904
- Q15: value MMBT3904 -> PZT2222A; footprint IPC-semi-nominal:SOT-23 -> IPC-semi-nominal:SOT-223
- Q17: value MMBT2907A -> TIP105; footprint IPC-semi-nominal:SOT-23 -> conn:CONN_3-SIL
- Q2: value MMBT3906 -> MMBT3904
- Q5: value PMP5201Y -> MMBT3906; footprint IPC-semi-nominal:SC-70-6 -> IPC-semi-nominal:SOT-23
- R10: renamed from R11; value 560 -> 470
- R11: renamed from R6; value 12k -> 100k
- R12: renamed from R8; value 62k 1% -> 22k
- R13: renamed from R7; value 56k 1% -> 22k
- R14: value 1k -> 22k 0.5%
- R2: value 4k7 -> 22k
- R21: renamed from R16; value 1k -> 22k
- R22: renamed from R17; value 150 -> 1k
- R23: renamed from R18; value 1k5 -> 22k
- R24: renamed from R20; value 12k -> 33
- R26: renamed from R22; value 1k -> 100k
- R27: renamed from R21; value 1k -> 22k
- R28: renamed from R25; value 10k -> 1k
- R29: renamed from R24; value 8k2 -> 1k
- R3: value 22k -> 33
- R32: renamed from R19; value 820 -> 10k
- R34: renamed from R41; value 10k -> 22k
- R4: value 2k2 -> 22k
- R8: renamed from R1; value 22k -> 10k
- R9: renamed from R5; value 2k2 -> 470
- RV3: value 5k -> 10k; footprint passive:TRIM-R-BOURNS-TC33X-2 -> conn:CONN_3-SIL
- RV4: footprint conn:CONN_3-SIL -> passive:TRIM-R-BOURNS-TC33X-2
- moved G*** 95.8 mm to (176.0, 124.0) (x2)
- moved J1 78.6 mm to (221.0, 97.0), turned to 270 degrees
- moved R32 76.6 mm to (206.0, 92.0), turned to 270 degrees
- moved RV5 74.0 mm to (214.0, 93.0), turned to 90 degrees
- moved Q19 72.5 mm to (203.0, 92.0)
- moved R35 69.1 mm to (210.0, 93.0), turned to 90 degrees
- moved R22 68.7 mm to (168.5, 110.0), turned to 270 degrees
- moved C2 67.6 mm to (167.5, 78.0)
- moved RV6 66.6 mm to (214.0, 101.0), turned to 270 degrees
- moved R23 66.5 mm to (172.0, 110.0), turned to 90 degrees
- moved D2 63.7 mm to (142.5, 76.5)
- moved R39 62.8 mm to (220.0, 81.0)
- moved D11 62.3 mm to (220.0, 84.0), turned to 0 degrees
- moved R36 62.1 mm to (210.0, 101.0), turned to 270 degrees
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- renumbered C5 to C7, C10 to C8, D8 to D9, DZ3 to DZ2, Q9 to Q10, Q6 to Q11, Q7 to Q12, Q12 to Q19, Q18 to Q3, Q4 to Q8, R10 to R15, R13 to R18, R23 to R31, R34 to R33, R30 to R37, R31 to R38, R32 to R39, R33 to R40, RV2 to RV1, RV1 to RV2
Connections:
- C1 pad 1: /VCC -> V+
- C1 pad 2: /V- -> V-UNREG
- C2 pad 1: /V+ -> GND
- C2 pad 2: /V- -> V-UNREG
- C3 pad 1: /V+ -> Net-(C3-Pad1)
- C6 pad 1: /FB- -> GND
- C6 pad 2: Net-(C6-Pad2) -> V-
- C7 pad 1: /V+ -> GND
- C8 pad 1: /V+ -> /OUT+
- C8 pad 2: Net-(C10-Pad2) -> /OUT-
- C9 pad 2: /VEE -> V-
- D1 pad 1: /V- -> Net-(D1-Pad1)
- D1 pad 2: Net-(D1-Pad2) -> V-UNREG
- D10 pad 1: Net-(D10-Pad1) -> /GUARD
- D10 pad 3: Net-(C6-Pad2) -> /FB-
- D11 pad 1: Net-(D14-Pad1) -> /OUT-
- D11 pad 2: Net-(C10-Pad2) -> Net-(D11-Pad2)
- D12 pad 2: /V+ -> /OUT+
- D2 pad 1: /VCC -> V+
- D2 pad 2: Net-(D1-Pad2) -> Net-(D1-Pad1)
- D3 pad 1: /VCC -> Net-(D3-Pad1)
- D3 pad 2: Net-(D1-Pad3) -> V-UNREG
- D5 pad 2: /VCC -> V+
- D7 pad 1: /V+ -> GND
- D8 pad 1: /VCC -> V+
- D8 pad 2: /V+ -> GND
- D9 pad 1: /V+ -> GND
- DS1 pad A: Net-(DS2-PadA) -> Net-(DS1-PadA)
- DS1 pad K: Net-(DS2-PadK) -> V-
- DZ1 pad 1: Net-(C4-Pad2) -> Net-(DZ1-Pad1)
- DZ2 pad A: Net-(C10-Pad2) -> /OUT-
- DZ2 pad K: /V+ -> /OUT+
- J1 pad 1: Net-(J1-Pad1) -> /OUT+
- J1 pad 2: Net-(C10-Pad2) -> Net-(J1-Pad2)
- J1 pad 3: Net-(J1-Pad3) -> /OUT-
- J1 pad 4: Net-(C8-Pad2) -> Net-(J1-Pad4)
- J3 pad 1: Net-(D1-Pad2) -> Net-(D1-Pad1)
- J4 pad 1: /V- -> V-UNREG
- J5 pad 1: Net-(D1-Pad3) -> Net-(D3-Pad1)
- J8 pad 1: /V+ -> /OUT+
- J9 pad 1: Net-(C10-Pad2) -> /OUT-
- Q1 pad 1: Net-(C3-Pad2) -> Net-(Q1-Pad1)
- Q1 pad 2: Net-(Q1-Pad2) -> V+
- Q1 pad 3: Net-(Q1-Pad3) -> Net-(C3-Pad1)
- Q10 pad 1: Net-(D10-Pad1) -> Net-(Q10-Pad1)
- Q10 pad 2: Net-(Q10-Pad1) -> V+
- Q10 pad 3: /V- -> Net-(Q10-Pad3)
- Q11 pad 1: /FB+ -> /FB-
- Q11 pad 2: /FB- -> /FB+
- Q11 pad 3: Net-(Q5-Pad1) -> Net-(Q11-Pad3)
- Q11 pad 4: Net-(D9-Pad1) -> /GUARD
- Q11 pad 5: Net-(D9-Pad1) -> /GUARD
- Q11 pad 6: Net-(Q6-Pad6) -> Net-(Q11-Pad6)
- Q12 pad 3: Net-(D9-Pad1) -> /GUARD
- Q13 pad 1: Net-(C8-Pad1) -> Net-(Q11-Pad6)
- Q13 pad 3: Net-(D13-Pad1) -> Net-(Q13-Pad3)
- Q14 pad 1: /VBIAS -> Net-(Q13-Pad3)
- Q14 pad 2: Net-(Q11-Pad2) -> Net-(Q14-Pad2)
- Q14 pad 3: Net-(Q11-Pad3) -> Net-(Q14-Pad3)
- Q15 pad 2: Net-(D13-Pad1) -> GND
- Q15 pad 3: Net-(DS2-PadK) -> Net-(Q15-Pad3)
- Q16 pad 1: Net-(C9-Pad1) -> Net-(Q15-Pad3)
- Q16 pad 2: /VEE -> /OUT-
- Q16 pad 3: Net-(Q16-Pad3) -> Net-(Q15-Pad1)
- Q17 pad 1: Net-(Q16-Pad3) -> Net-(Q14-Pad3)
- Q17 pad 2: Net-(DS1-PadK) -> V-UNREG
- Q17 pad 3: Net-(C9-Pad1) -> /OUT-
- Q19 pad 1: /VBIAS -> Net-(Q19-Pad1)
- Q19 pad 2: Net-(Q12-Pad2) (its old number) -> V+
- Q19 pad 3: Net-(Q12-Pad3) -> Net-(Q19-Pad3)
- Q2 pad 1: Net-(C11-Pad1) -> Net-(Q2-Pad1)
- Q2 pad 2: Net-(Q1-Pad2) -> V-UNREG
- Q2 pad 3: /V- -> Net-(Q2-Pad3)
- Q3 pad 1: Net-(Q1-Pad3) -> Net-(C3-Pad2)
- Q3 pad 2: /VEE -> V-
- Q3 pad 3: Net-(Q18-Pad3) -> Net-(Q2-Pad1)
- Q3 pad 4: /VEE -> V-
- Q5 pad 2: Net-(Q5-Pad1) -> V+
- Q8 pad 1: /V+ -> GND
- Q8 pad 3: /V+ -> V+
- Q8 pad 5: Net-(Q4-Pad5) -> Net-(Q8-Pad5)
- Q8 pad 6: /V+ -> V+
- R10 pad 2: /VEE -> V-
- R11 pad 1: /V+ -> GND
- R12 pad 1: Net-(Q4-Pad5) -> Net-(Q8-Pad5)
- R12 pad 2: /VEE -> V-
- R13 pad 2: /VEE -> V-
- R14 pad 1: Net-(Q5-Pad6) -> Net-(Q8-Pad5)
- R14 pad 2: Net-(Q6-Pad6) -> /FB-
- R18 pad 2: /VEE -> V-
- R2 pad 1: Net-(Q1-Pad3) -> Net-(C3-Pad2)
- R2 pad 2: /V- -> Net-(Q2-Pad3)
- R21 pad 1: Net-(C8-Pad2) -> V+
- R21 pad 2: Net-(Q10-Pad1) -> Net-(Q14-Pad3)
- R22 pad 1: /VBIAS -> Net-(Q14-Pad2)
- R22 pad 2: /V+ -> V-UNREG
- R23 pad 1: /VCC -> Net-(Q15-Pad1)
- R23 pad 2: Net-(Q11-Pad2) -> Net-(Q14-Pad3)
- R24 pad 1: Net-(C8-Pad1) -> /OUT-
- R24 pad 2: Net-(C8-Pad2) -> Net-(Q15-Pad3)
- R26 pad 1: Net-(Q14-Pad1) -> GND
- R26 pad 2: Net-(D13-Pad1) -> Net-(Q18-Pad1)
- R27 pad 1: Net-(Q13-Pad6) -> Net-(R27-Pad1)
- R27 pad 2: Net-(Q14-Pad1) -> Net-(R27-Pad2)
- R28 pad 1: Net-(Q13-Pad2) -> Net-(Q20-Pad1)
- R28 pad 2: Net-(C10-Pad2) -> Net-(Q18-Pad6)
- R29 pad 1: /V+ -> V+
- R29 pad 2: Net-(DS2-PadA) -> Net-(Q20-Pad1)
- R3 pad 1: /V+ -> Net-(Q2-Pad1)
- R3 pad 2: Net-(Q1-Pad2) -> V-UNREG
- R31 pad 1: Net-(Q13-Pad6) -> Net-(Q18-Pad6)
- R31 pad 2: Net-(Q15-Pad1) -> Net-(Q19-Pad1)
- R32 pad 1: /VCC -> Net-(Q19-Pad3)
- R32 pad 2: Net-(Q12-Pad2) (its old number) -> Net-(DS1-PadA)
- R33 pad 1: Net-(C8-Pad2) -> GND
- R33 pad 2: Net-(C10-Pad2) -> /OUT+
- R34 pad 1: /V+ -> /OUT+
- R34 pad 2: Net-(C10-Pad2) -> /OUT-
- R35 pad 1: Net-(C10-Pad2) -> GND
- R36 pad 1: /V+ -> /OUT+
- R38 pad 1: Net-(D14-Pad1) -> Net-(D11-Pad2)
- R39 pad 1: Net-(C10-Pad2) -> /OUT-
- R39 pad 2: Net-(D14-Pad1) -> Net-(D11-Pad2)
- R4 pad 1: Net-(C4-Pad2) -> Net-(Q1-Pad1)
- R4 pad 2: Net-(R4-Pad2) -> V-
- R40 pad 1: /V+ -> /OUT+
- R8 pad 1: Net-(C4-Pad2) -> Net-(DZ1-Pad1)
- R8 pad 2: Net-(C3-Pad2) -> Net-(C5-Pad2)
- R9 pad 1: Net-(R4-Pad2) -> Net-(DZ1-Pad1)
- RV1 pad 1: /V+ -> GND
- RV2 pad 2: Net-(C4-Pad2) -> Net-(DZ1-Pad1)
- RV2 pad 3: Net-(C4-Pad2) -> Net-(DZ1-Pad1)
- RV3 pad 1: Net-(C8-Pad2) -> GND
- RV3 pad 2: Net-(RV3-Pad2) -> Net-(Q18-Pad1)
- RV3 pad 3: Net-(Q11-Pad3) -> Net-(R27-Pad1)
- RV4 pad 1: Net-(RV3-Pad2) -> Net-(R27-Pad2)
- RV4 pad 2: Net-(C8-Pad1) -> V-
- RV4 pad 3: Net-(C8-Pad2) -> V-
- RV5 pad 1: Net-(R35-Pad2) -> Net-(J1-Pad2)
- RV5 pad 2: Net-(J1-Pad3) -> Net-(J1-Pad2)
- RV5 pad 3: Net-(J1-Pad3) -> Net-(R35-Pad2)
- RV6 pad 1: Net-(R36-Pad2) -> Net-(J1-Pad4)
- RV6 pad 2: Net-(J1-Pad1) -> Net-(J1-Pad4)
- RV6 pad 3: Net-(J1-Pad1) -> Net-(R36-Pad2)
Routing:
- net /V+: track 931.2 -> 0.00 mm, vias 48 -> 0
- net CGND: track 0.00 -> 404.7 mm, vias 0 -> 29
- net GND: track 0.00 -> 357.8 mm, vias 0 -> 22
- net V-: track 0.00 -> 287.5 mm, vias 0 -> 11
- net V+: track 0.00 -> 252.6 mm, vias 0 -> 9
- net /V-: track 201.0 -> 0.00 mm, vias 1 -> 0
- net /OUT+: track 0.00 -> 195.2 mm
- net Net-(C10-Pad2): track 191.7 -> 0.00 mm
- net V-UNREG: track 0.00 -> 183.5 mm, vias 0 -> 1
- net /VEE: track 164.3 -> 0.00 mm, vias 16 -> 0
- net /OUT-: track 0.00 -> 141.6 mm
- net /VCC: track 134.6 -> 0.00 mm, vias 2 -> 0
- net (no net): track 120.0 -> 0.00 mm
- net Net-(C8-Pad2): track 82.0 -> 0.00 mm
- net Net-(D1-Pad3): track 47.2 -> 0.00 mm
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- added copper zone on F.Cu, net /OUT+
- added copper zone on F.Cu, net /OUT-
- added copper zone on B.Cu, net CGND
- added copper zone on F.Cu, net CGND
- added copper zone on B.Cu, net GND
- added copper zone on F.Cu, net GND
- added copper zone on F.Cu, net Net-(D1-Pad1)
- added copper zone on F.Cu, net Net-(D3-Pad1)
- added copper zone on B.Cu, net V+
- added copper zone on F.Cu, net V+
- added copper zone on B.Cu, net V-
- added copper zone on F.Cu, net V-
- added copper zone on B.Cu, net V-UNREG
- added copper zone on F.Cu, net V-UNREG
- removed copper zone on B.Cu, net /V+
- removed copper zone on F.Cu, net /V+
- removed copper zone on B.Cu, net /VEE
- removed copper zone on F.Cu, net /VEE
- removed copper zone on F.Cu, net Net-(D9-Pad3)
Other:
- board size 100 x 100 mm -> 100 x 75 mm
- board text added: "+"
- board text added: "-"
- board text added: "CURRENT LIMITER"
- board text added: "ERROR AMPL."
- board text added: "FEEDBACK INPUT"
- board text added: "GND"
- board text added: "LOCAL REGULATOR"
- board text added: "OUTPUT FILTER"
- board text added: "POWER INPUT"
- board text added: "Rev C Mar 2014"
- board text added: "VOLTAGE REFERENCE"
- board text removed: "-OUT+"
- board text removed: "-SENSE+"
- board text removed: "CURR"
- board text removed: "CURRENT"
- board text removed: "CURRENT ERROR AMP"
- board text removed: "CURRENT REFERENCE AND BIAS"
- board text removed: "HOT"
- board text removed: "LIMIT"
- board text removed: "MAX CURR TRIM"
- board text removed: "MAX VOLT TRIM"
- board text removed: "METER"
- board text removed: "REFERENCE and LOCAL REGULATOR"
- board text removed: "Rev B Jan 2014"
- board text removed: "SETPOINT SELECTOR and BUFFER"
- board text removed: "T SENSE"
- board text removed: "VOLT"
- board text removed: "VOLTAGE ERROR AMP"
- board text removed: "c4757p JAN 2014 PS-1 rB"

Commit message: Few BOM-related changes
Parts:
- removed R2: 22k, IPC7351-Nominal:RESC2012X50
Connections:
- net /GUARD renamed Net-(D10-Pad1)
- Q2 pad 3: Net-(Q2-Pad3) -> Net-(C3-Pad2)
Routing:
- net Net-(C3-Pad2): track 7.31 -> 18.7 mm
- net Net-(Q2-Pad3): track 8.51 -> 0.00 mm
