File: Proj-Main/psu.sch (KiCad schematic (older format))
At the start: 127 parts, among them J1 T1A, J2 T1B, J3 T1C, J4 OUT+, J5 SENSE, J6 METER, J7 OUT-, Q1 BC856, Q10 PMP4201Y, Q11 MMBT3904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

Commit message: PCB REV A
Connections:
- wire segments 433 -> 309
Other:
- note added: "REFERENCE"
- note removed: "OUTPUT FILTER"
- note removed: "VOLTAGE REFERENCE"
- moved on the sheet: C2, C4
